File: displayBoard.kicad_sch (KiCad schematic)
At the start: 15 parts, among them J1 FPC, J2 USB_C, J3 BNO085, J4 NEO_M9N, U1 STM32U599VJTx

Commit message: Se actualizan los esquemas para botones, leds de status y leds de direccionables
Parts:
- added C10, C11, C12, C13, C14, C15, C16, C17, C18, C19, C20, C21, C22, C23, C24, C25, C26: 100nF, symbol Device:C_Small
- added D10, D11, D12, D13, D14, D15, D2, D3, D4, D5, D6, D7, D8, D9: APA102, LED_SMD:LED_RGB_5050-6, symbol LED:APA102
- added D16: YELLOW, symbol Device:LED_Small
- added D17: BLUE, symbol Device:LED_Small
- added R1: 10K, symbol Device:R_Small
- added R2, R3, R4, R5: 4.7K, symbol Device:R_Small
- added SW1, SW2: SW_Push_Dual_x2, symbol Switch:SW_Push_Dual_x2
Connections:
- net +3.3V: now also D1.4 (VCC), J1.4 (Pin_4), J3.1 (Pin_1), J3.10 (Pin_10), J3.9 (Pin_9), J4.1 (Pin_1), C10.1, C11.1, C12.1, C13.1, C14.1, C15.1, C16.1, C17.1, C18.1, C19.1, C20.1, C21.1, C22.1, C23.1, C24.1, D10.4 (VCC), D11.4 (VCC), D12.4 (VCC), D13.4 (VCC), D14.4 (VCC), D15.4 (VCC), D2.4 (VCC), D3.4 (VCC), D4.4 (VCC), D5.4 (VCC), D6.4 (VCC), D7.4 (VCC), D8.4 (VCC), D9.4 (VCC), R1.1, R2.1, R5.1, SW1.2 (D)
- net BNO085_CS: now also J3.6 (Pin_6)
- net BNO085_INT: now also J3.7 (Pin_7), U1.88 (PD7); no longer U1.68 (PA9)
- net BNO085_MISO: now also J3.4 (Pin_4), U1.90 (PB4); no longer U1.79 (PC11)
- net BNO085_MOSI: now also J3.5 (Pin_5), U1.91 (PB5); no longer U1.80 (PC12)
- net BNO085_SCK: now also J3.3 (Pin_3), U1.89 (PB3); no longer U1.78 (PC10)
- net BUTTON_BACK: now also U1.7 (PC13); no longer U1.29 (PA4)
- net BUTTON_DOWN: now also U1.51 (PB12); no longer U1.34 (PC5)
- net BUTTON_NEXT: now also U1.29 (PA4); no longer U1.31 (PA6)
- net BUTTON_OK: now also U1.34 (PC5); no longer U1.33 (PC4)
- net BUTTON_SETTINGS: now also U1.33 (PC4); no longer U1.30 (PA5)
- net BUTTON_UP: now also U1.30 (PA5); no longer U1.32 (PA7)
- net GND: now also D1.3 (GND), J1.29 (Pin_29), J1.3 (Pin_3), J1.36 (Pin_36), J3.2 (Pin_2), J4.4 (Pin_4), U1.20 (VREF-), C10.2, C11.2, C12.2, C13.2, C14.2, C15.2, C16.2, C17.2, C18.2, C19.2, C20.2, C21.2, C22.2, C23.2, C24.2, C25.2, C26.2, D10.3 (GND), D11.3 (GND), D12.3 (GND), D13.3 (GND), D14.3 (GND), D15.3 (GND), D16.1 (K), D17.1 (K), D2.3 (GND), D3.3 (GND), D4.3 (GND), D5.3 (GND), D6.3 (GND), D7.3 (GND), D8.3 (GND), D9.3 (GND), R4.2, SW2.1 (C)
- net LTDC_B0: now also J1.21 (Pin_21)
- net LTDC_B1: now also J1.22 (Pin_22)
- net LTDC_B2: now also J1.23 (Pin_23)
- net LTDC_B3: now also J1.24 (Pin_24)
- net LTDC_B4: now also J1.25 (Pin_25)
- net LTDC_B5: now also J1.26 (Pin_26)
- net LTDC_B6: now also J1.27 (Pin_27)
- net LTDC_B7: now also J1.28 (Pin_28)
- net LTDC_CLK: now also J1.30 (Pin_30)
- net LTDC_DE: now also J1.34 (Pin_34)
- net LTDC_G0: now also J1.13 (Pin_13)
- net LTDC_G1: now also J1.14 (Pin_14)
- net LTDC_G2: now also J1.15 (Pin_15)
- net LTDC_G3: now also J1.16 (Pin_16)
- net LTDC_G4: now also J1.17 (Pin_17)
- net LTDC_G5: now also J1.18 (Pin_18)
- net LTDC_G6: now also J1.19 (Pin_19)
- net LTDC_G7: now also J1.20 (Pin_20)
- net LTDC_HSYNC: now also J1.32 (Pin_32)
- net LTDC_R0: now also J1.5 (Pin_5)
- net LTDC_R1: now also J1.6 (Pin_6)
- net LTDC_R2: now also J1.7 (Pin_7)
- net LTDC_R3: now also J1.8 (Pin_8)
- net LTDC_R4: now also J1.9 (Pin_9)
- net LTDC_R5: now also J1.10 (Pin_10)
- net LTDC_R6: now also J1.11 (Pin_11)
- net LTDC_R7: now also J1.12 (Pin_12)
- net LTDC_VSYNC: now also J1.33 (Pin_33)
- net NEO_M9N_RX: now also J4.3 (Pin_3), U1.24 (PA1); no longer U1.17 (PC2)
- net NEO_M9N_TX: now also J4.2 (Pin_2), U1.23 (PA0); no longer U1.18 (PC3)
- net NRST: now reaches U1.14 (NRST)
- net NRST: now also C26.1, R5.2, SW2.2 (D)
- net PSRAM_IO7: now reaches U1.15 (PC0)
- net PSRAM_IO4: now reaches U1.16 (PC1)
- net 3.3V: now reaches U1.21 (VREF+)
- net PSRAM_NCS: now reaches U1.25 (PA2)
- net PSRAM_CLK: now reaches U1.26 (PA3)
- net PSRAM_IO1: now reaches U1.35 (PB0)
- net PSRAM_IO0: now reaches U1.36 (PB1)
- net PB10: now reaches U1.47 (PB10)
- net STATUS_LED: now reaches U1.53 (PB14)
- net STATUS_LED: now also R3.1
- net PC6: now reaches U1.63 (PC6)
- net SDMMC_CK: now reaches U1.64 (PC7)
- net SDMMC_D0: now reaches U1.65 (PC8)
- net SDMMC_D1: now reaches U1.66 (PC9)
- net PA8: now reaches U1.67 (PA8)
- net SDMMC_CMD: now reaches U1.83 (PD2)
- net PD4: now reaches U1.85 (PD4)
- net PSRAM_IO5: now reaches U1.86 (PD5)
- net BOOT0: now reaches U1.94 (PH3)
- net BOOT0: now also C25.1, R4.1, SW1.1 (C)
- net BNO085_RST: now reaches U1.95 (PB8)
- net BNO085_RST: now also J3.8 (Pin_8)
- net PB9: now reaches U1.96 (PB9)
- net PE1: now reaches U1.98 (PE1)
- net LEDK: now reaches J1.1 (Pin_1)
- net LEDA: now reaches J1.2 (Pin_2)
- net DISP: now reaches J1.31 (Pin_31)
- net DISP: now also R1.2
- net at D1.5 (CO): now also D2.2 (CI)
- net at D1.6 (DO): now also D2.1 (DI)
- new net: D5.6 (DO), D6.1 (DI)
- new net: D5.5 (CO), D6.2 (CI)
- new net: D6.5 (CO), D7.2 (CI)
- new net: D6.6 (DO), D7.1 (DI)
- new net: D4.6 (DO), D5.1 (DI)
- new net: D4.5 (CO), D5.2 (CI)
- new net: D2.5 (CO), D3.2 (CI)
- new net: D2.6 (DO), D3.1 (DI)
- new net: D7.5 (CO), D8.2 (CI)
- new net: D7.6 (DO), D8.1 (DI)
- new net: D3.6 (DO), D4.1 (DI)
- new net: D3.5 (CO), D4.2 (CI)
- new net: D17.2 (A), R3.2
- new net: D14.6 (DO), D15.1 (DI)
- new net: D14.5 (CO), D15.2 (CI)
- new net: D11.6 (DO), D12.1 (DI)
- new net: D11.5 (CO), D12.2 (CI)
- new net: D12.5 (CO), D13.2 (CI)
- new net: D12.6 (DO), D13.1 (DI)
- new net: D10.6 (DO), D11.1 (DI)
- new net: D10.5 (CO), D11.2 (CI)
- new net: D16.2 (A), R2.2
- new net: D8.5 (CO), D9.2 (CI)
- new net: D8.6 (DO), D9.1 (DI)
- new net: D10.2 (CI), D9.5 (CO)
- new net: D10.1 (DI), D9.6 (DO)
- new net: D13.6 (DO), D14.1 (DI)
- new net: D13.5 (CO), D14.2 (CI)
- new net PA9: U1.68 (PA9)
- new net PC12: U1.80 (PC12)
- new net PC2: U1.17 (PC2)
- new net PSRAM_IO2: U1.32 (PA7)
- new net PSRAM_IO3: U1.31 (PA6)
- new net PSRAM_IO6: U1.18 (PC3)
- new net SDMMC_D2: U1.78 (PC10)
- new net SDMMC_D3: U1.79 (PC11)
- no-connect marks 0 -> 5
Other:
- company: (none) -> Oublik
- title: (none) -> lapTimer devBoard
- moved on the sheet: D1, J1, J2, J3, J4, U1
